File: hardware/kicad/MicroKeyboard.kicad_pcb (KiCad board)
At the start: 2 copper layers, 0 parts

Commit message: 昇圧モジュールとXIAO nRF52840のKiCad部品を追加
- シンボル・フットプリント・3Dモデルを登録
- 回路図とPCBに各モジュールを配置
- 部品表・寸法資料・モデルの出典を追加
Parts:
- added U1: AE-XCL103-3V3, micro_keyboard:AE-XCL103-3V3_Horizontal, F.Cu at (89.0, 90.0)
- added U2: XIAO nRF52840, micro_keyboard:XIAO-nRF52840-SMD, F.Cu at (105.0, 100.0)
