File: hardware/kicad/MicroKeyboard.kicad_sch (KiCad schematic)
At the start: 0 parts

Commit message: 昇圧モジュールとXIAO nRF52840のKiCad部品を追加
- シンボル・フットプリント・3Dモデルを登録
- 回路図とPCBに各モジュールを配置
- 部品表・寸法資料・モデルの出典を追加
Parts:
- added U1: AE-XCL103-3V3, micro_keyboard:AE-XCL103-3V3_Horizontal, symbol micro_keyboard:AE-XCL103-3V3
- added U2: XIAO nRF52840, micro_keyboard:XIAO-nRF52840-SMD, symbol micro_keyboard:XIAO-nRF52840-SMD
Other:
- note added: "制御モジュール（表面実装）"
- note added: "昇圧モジュール（平置き・直ピン）"
